File: cpu-fast.brd (EAGLE design)
At the start: 25.4 x 25.4 mm, 14 parts, among them IC1 PIC18F4550_QFN, Y2 20Mhz

Commit message: Changes I forgot to commit
Parts:
- added C2: 0.47uF, SparkFun-Capacitors:0603-CAP
- R1: value (none) -> 1k
Connections:
- net RESET renamed MCLR
- new net N$7: C2.1, IC1.37
- net GND: now also C2.2
Routing:
- net GND: track 42.6 -> 48.8 mm
- net N$7: track 0.00 -> 1.56 mm
Changed lines of the file:
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@@
 <attribute name="NAME" x="20.3975" y="20.43125" size="1.016" layer="25" rot="R90"/>
 </element>
-<element name="R1" library="SparkFun-Passives" package="0402-RES" value="" x="20.79625" y="13.6525" rot="R180"/>
+<element name="R1" library="SparkFun-Passives" package="0402-RES" value="1k" x="20.79625" y="13.6525" rot="R180"/>
 <element name="JP2" library="SparkFun-Connectors" package="1X08" value="" x="1.42875" y="3.81" smashed="yes" rot="R90">
 <attribute name="VALUE" x="4.60375" y="2.54" size="1.27" layer="27" rot="R90"/>
@@
 <element name="Y2" library="SparkFun-FreqCtrl" package="RESONATOR-SMD" value="20Mhz" x="12.85875" y="14.44625" rot="R135">
 <attribute name="PROD_ID" value="XTAL-08900" x="12.85875" y="14.44625" size="1.778" layer="27" rot="R135" display="off"/>
+</element>
+<element name="C2" library="SparkFun-Capacitors" package="0603-CAP" value="0.47uF" x="7.46125" y="13.97" rot="R135">
+<attribute name="PROD_ID" value="CAP-07822" x="7.46125" y="13.97" size="1.778" layer="27" rot="R135" display="off"/>
 </element>
 </elements>
@@
 <wire x1="9.525" y1="21.59" x2="9.525" y2="22.38375" width="0.4064" layer="16"/>
 <wire x1="11.1584375" y1="3.897103125" x2="11.563040625" y2="3.4925" width="0.254" layer="1"/>
-<wire x1="11.563040625" y1="3.4925" x2="13.0175" y2="3.4925" width="0.254" layer="1"/>
-<via x="13.0175" y="3.4925" extent="1-16" drill="0.6"/>
-<wire x1="13.0175" y1="3.4925" x2="13.6525" y2="3.4925" width="0.254" layer="16"/>
+<wire x1="11.563040625" y1="3.4925" x2="14.9225" y2="3.4925" width="0.254" layer="1"/>
+<via x="14.9225" y="3.4925" extent="1-16" drill="0.6"/>
+<wire x1="14.9225" y1="3.4925" x2="13.6525" y2="3.4925" width="0.254" layer="16"/>
 <wire x1="11.1584375" y1="3.897103125" x2="10.31875" y2="4.736790625" width="0.254" layer="1"/>
 <wire x1="15.875" y1="11.9895" x2="17.4625" y2="11.9895" width="0.254" layer="1"/>
@@
 <wire x1="12.099328125" y1="11.9895" x2="12.492328125" y2="12.3825" width="0.254" layer="1"/>
 <wire x1="12.492328125" y1="12.3825" x2="15.08125" y2="12.3825" width="0.254" layer="1"/>
+<contactref element="C2" pad="2"/>
+<wire x1="6.86020625" y1="14.571040625" x2="6.50875" y2="14.922496875" width="0.254" layer="1"/>
+<wire x1="6.50875" y1="14.922496875" x2="6.50875" y2="15.875" width="0.254" layer="1"/>
+<wire x1="6.50875" y1="15.875" x2="7.925" y2="17.29125" width="0.254" layer="1"/>
+<wire x1="7.925" y1="17.29125" x2="7.925" y2="17.526" width="0.254" layer="1"/>
 </signal>
 <signal name="+5V">
@@
 <wire x1="11.2918" y1="14.57635625" x2="10.95375" y2="14.23830625" width="0.254" layer="1"/>
 </signal>
-<signal name="RESET">
+<signal name="MCLR">
 <contactref element="IC1" pad="18"/>
 <contactref element="R1" pad="1"/>
 <contactref element="JP1" pad="6"/>
-<wire x1="13.456534375" y1="6.1952" x2="16.476734375" y2="3.175" width="0.254" layer="1"/>
-<wire x1="16.476734375" y1="3.175" x2="18.7325" y2="3.175" width="0.254" layer="1"/>
-<wire x1="18.7325" y1="3.175" x2="20.0025" y2="4.445" width="0.254" layer="1"/>
-<wire x1="20.0025" y1="4.445" x2="20.0025" y2="6.985" width="0.254" layer="1"/>
-<wire x1="20.0025" y1="6.985" x2="19.84375" y2="7.14375" width="0.254" layer="1"/>
-<wire x1="19.84375" y1="7.14375" x2="19.84375" y2="9.8425" width="0.254" layer="1"/>
 <wire x1="19.84375" y1="9.8425" x2="22.225" y2="12.22375" width="0.254" layer="1"/>
 <wire x1="22.225" y1="12.22375" x2="22.225" y2="13.6525" width="0.254" layer="1"/>
@@
 <wire x1="23.495" y1="16.51" x2="23.97125" y2="16.51" width="0.254" layer="1"/>
 <wire x1="21.44625" y1="13.6525" x2="22.225" y2="13.6525" width="0.254" layer="1"/>
+<wire x1="19.84375" y1="9.8425" x2="19.84375" y2="4.28625" width="0.254" layer="1"/>
+<wire x1="19.84375" y1="4.28625" x2="18.89125" y2="3.33375" width="0.254" layer="1"/>
+<wire x1="18.89125" y1="3.33375" x2="16.317984375" y2="3.33375" width="0.254" layer="1"/>
+<wire x1="16.317984375" y1="3.33375" x2="13.456534375" y2="6.1952" width="0.254" layer="1"/>
 </signal>
 <signal name="IO5">
@@
 <wire x1="9.8425" y1="2.69875" x2="19.05" y2="2.69875" width="0.254" layer="1"/>
 <wire x1="19.05" y1="2.69875" x2="20.47875" y2="4.1275" width="0.254" layer="1"/>
-<wire x1="20.47875" y1="4.1275" x2="20.47875" y2="7.3025" width="0.254" layer="1"/>
-<wire x1="20.47875" y1="7.3025" x2="20.32" y2="7.46125" width="0.254" layer="1"/>
-<wire x1="20.32" y1="7.46125" x2="20.32" y2="9.525" width="0.254" layer="1"/>
+<wire x1="20.47875" y1="4.1275" x2="20.47875" y2="7.9375" width="0.254" layer="1"/>
+<wire x1="20.32" y1="8.09625" x2="20.32" y2="9.525" width="0.254" layer="1"/>
 <wire x1="20.32" y1="9.525" x2="22.70125" y2="11.90625" width="0.254" layer="1"/>
 <wire x1="22.70125" y1="11.90625" x2="22.70125" y2="12.54125" width="0.254" layer="1"/>
 <wire x1="22.70125" y1="12.54125" x2="23.97125" y2="13.81125" width="0.254" layer="1"/>
 <wire x1="23.97125" y1="13.81125" x2="23.97125" y2="13.97" width="0.254" layer="1"/>
+<wire x1="20.47875" y1="7.9375" x2="20.32" y2="8.09625" width="0.254" layer="1"/>
 </signal>
 <signal name="N$4">
@@
 <contactref element="IC1" pad="15"/>
 </signal>
+<signal name="N$7">
+<contactref element="IC1" pad="37"/>
+<contactref element="C2" pad="1"/>
+<wire x1="8.559821875" y1="12.011153125" x2="8.062290625" y2="12.508684375" width="0.254" layer="1"/>
+<wire x1="8.062290625" y1="12.508684375" x2="8.062290625" y2="13.36895625" width="0.254" layer="1"/>
+</signal>
 </signals>
