File: cpu-fast.sch (EAGLE design)
At the start: 14 parts, among them IC1 PIC18F4550_QFN, Y2 20Mhz

Commit message: Changes I forgot to commit
Parts:
- added C2: 0.47uF, SparkFun-Capacitors:0.22UF-25V-10%(0603)
- R1: value (none) -> 1k
Connections:
- net RESET renamed MCLR
- new net N$7: C2.1, IC1.VUSB
- net GND: now also C2.2
Changed lines of the file:
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@@
 <part name="P+1" library="supply1" deviceset="+5V" device=""/>
 <part name="C1" library="rcl" deviceset="C-EU" device="C0805K" value="470n"/>
-<part name="R1" library="SparkFun-Passives" deviceset="RESISTOR" device="0402-RES"/>
+<part name="R1" library="SparkFun-Passives" deviceset="RESISTOR" device="0402-RES" value="1k"/>
 <part name="P+2" library="supply1" deviceset="+5V" device=""/>
 <part name="JP2" library="SparkFun-Connectors" deviceset="M08" device="1X08"/>
@@
 <part name="GND5" library="supply1" deviceset="GND" device=""/>
 <part name="Y2" library="SparkFun-FreqCtrl" deviceset="RESONATOR" device="16MHZ" value="20Mhz"/>
+<part name="C2" library="SparkFun-Capacitors" deviceset="0.22UF-25V-10%(0603)" device="" value="0.47uF"/>
 </parts>
 <sheets>
@@
 <instance part="GND5" gate="1" x="208.28" y="73.66"/>
 <instance part="Y2" gate="G$1" x="208.28" y="86.36"/>
+<instance part="C2" gate="G$1" x="233.68" y="137.16"/>
 </instances>
 <busses>
@@
 <pinref part="IC1" gate="G$1" pin="VSS@1"/>
 <wire x1="203.2" y1="129.54" x2="226.06" y2="129.54" width="0.1524" layer="91"/>
-<wire x1="226.06" y1="129.54" x2="226.06" y2="104.14" width="0.1524" layer="91"/>
+<wire x1="226.06" y1="129.54" x2="226.06" y2="109.22" width="0.1524" layer="91"/>
 <pinref part="IC1" gate="G$1" pin="VSS@2"/>
+<wire x1="226.06" y1="109.22" x2="226.06" y2="104.14" width="0.1524" layer="91"/>
 <wire x1="203.2" y1="132.08" x2="226.06" y2="132.08" width="0.1524" layer="91"/>
 <wire x1="226.06" y1="132.08" x2="226.06" y2="129.54" width="0.1524" layer="91"/>
@@
 <label x="205.74" y="132.08" size="1.778" layer="95"/>
 <label x="205.74" y="129.54" size="1.778" layer="95"/>
+<pinref part="C2" gate="G$1" pin="2"/>
+<wire x1="233.68" y1="134.62" x2="233.68" y2="109.22" width="0.1524" layer="91"/>
+<wire x1="233.68" y1="109.22" x2="226.06" y2="109.22" width="0.1524" layer="91"/>
+<junction x="226.06" y="109.22"/>
 </segment>
 <segment>
@@
 </segment>
 </net>
-<net name="RESET" class="0">
+<net name="MCLR" class="0">
 <segment>
 <pinref part="IC1" gate="G$1" pin="!MCLR!/VPP/RE3"/>
@@
 </segment>
 </net>
+<net name="N$7" class="0">
+<segment>
+<pinref part="IC1" gate="G$1" pin="VUSB"/>
+<pinref part="C2" gate="G$1" pin="1"/>
+<wire x1="203.2" y1="147.32" x2="233.68" y2="147.32" width="0.1524" layer="91"/>
+<wire x1="233.68" y1="147.32" x2="233.68" y2="142.24" width="0.1524" layer="91"/>
+</segment>
+</net>
